Commit message: gazebo arms

File: rarms_gazebo/urdf/r2_arm.xacro (robot description, xacro)
@@ -6,5 +6,5 @@
     <!-- Constants for the robotic arm (masses in kg, lengths in m) -->
     <xacro:property name="max_effort" value="100" />
-    <xacro:property name="max_velocity" value="0.5" />
+    <xacro:property name="max_velocity" value="${M_PI/4}" />
     <xacro:property name="damping_1" value="0.02" />
     <xacro:property name="damping_2" value="0.02" />
@@ -15,5 +15,5 @@
     <!-- joint_f1 fixed -->
     <!-- link_1 -->
-    <xacro:property name="length_1" value="0.005" />
+    <xacro:property name="length_1" value="0.012" />
     <xacro:property name="radius_1" value="0.005" />
     <xacro:property name="mass_1" value="0.100" />
@@ -143,4 +143,9 @@
     </gazebo>
     </xacro:macro>
+    <xacro:macro name="gazebo_self_collision" params="link_name">
+    <gazebo reference="${link_name}">
+      <selfCollide>true</selfCollide>
+    </gazebo>
+    </xacro:macro>
     <!--=============================================================================-->
     <link name="world"/>
@@ -335,4 +340,12 @@
     </link>
     <xacro:gazebo_red_link_color_block link_name="link_ee"/>
+<!-- self collision -->
+     <xacro:gazebo_self_collision link_name="base_link"/>
+     <xacro:gazebo_self_collision link_name="link_1"/>
+     <xacro:gazebo_self_collision link_name="link_2"/>
+     <xacro:gazebo_self_collision link_name="link_3"/>
+     <xacro:gazebo_self_collision link_name="link_j1"/>
+     <xacro:gazebo_self_collision link_name="link_j2"/>
+     <xacro:gazebo_self_collision link_name="link_ee"/>
 <!-- ========================================================================= -->
     <!-- Transmissions for ros control -->

File: rarms_gazebo/urdf/r3_arm.xacro (robot description, xacro)
@@ -378,5 +378,4 @@
     <xacro:gazebo_grey_link_color_block link_name="link_4"/>
     <!-- fixed joint link_4 - link_ee -->
-    <!--
     <xacro:include filename="$(find rarms_gazebo)/urdf/hand.xacro" />
     <joint name="joint_f4" type="fixed">
@@ -389,7 +388,7 @@
         <preserveFixedJoint>true</preserveFixedJoint>
     </gazebo>
-    -->
+    <!-- fixed joint link_4 - EE_gripper -->
+<!--
     <xacro:include filename="$(find rarms_gazebo)/urdf/hand2.xacro" />
-    <!-- fixed joint link_4 - EE_gripper -->
     <joint name="joint_f4" type="fixed">
         <origin xyz="${0.0} ${length_EE_1/2} ${length_4+base_EE_1/2}" rpy="${M_PI/2} ${M_PI/2} 0.0"/>
@@ -401,6 +400,6 @@
         <preserveFixedJoint>true</preserveFixedJoint>
     </gazebo>
+-->
 <!-- self collision -->
-<!--
      <xacro:gazebo_self_collision link_name="base_link"/>
      <xacro:gazebo_self_collision link_name="link_1"/>
@@ -414,5 +413,4 @@
      <xacro:gazebo_self_collision link_name="EE_part_21"/>
      <xacro:gazebo_self_collision link_name="EE_part_22"/>
--->
 <!-- ========================================================================= -->
     <!-- Transmissions for ros control -->
